File: minimouse.kicad_pcb (KiCad board)
At the start: 2 copper layers, 90 x 85 mm, 22 parts, among them J1 Conn_ARM_JTAG_SWD_10, J5 Conn_01x02, M1 N20_encoder, M2 N20_encoder, U1 STM32F030C8Tx, U4 HC-SR04

Commit message: TP4
Parts:
- added C11: 2.2uF, Capacitor_SMD:C_0603_1608Metric, F.Cu at (179.5, 83.8)
- added C12: 2.2uF, Capacitor_SMD:C_0603_1608Metric, F.Cu at (170.6, 83.8)
- added C17: 2.2uF, Capacitor_SMD:C_0603_1608Metric, F.Cu at (153.8, 72.6)
- added C18: 2.2uF, Capacitor_SMD:C_0603_1608Metric, F.Cu at (121.3, 76.3)
- added C19: 2.2uF, Capacitor_SMD:C_0603_1608Metric, F.Cu at (172.5, 95.8)
- added C20: 2.2uF, Capacitor_SMD:C_0603_1608Metric, F.Cu at (127.6, 96.0)
- added C7: 2.2uF, Capacitor_SMD:C_0603_1608Metric, F.Cu at (150.0, 108.3)
- added C8: 0.1uF, Capacitor_SMD:C_0603_1608Metric, F.Cu at (156.7, 101.6)
- added C9: 22nF, Capacitor_SMD:C_0603_1608Metric, F.Cu at (158.2, 101.6)
- added D1: ON, LED_SMD:LED_0603_1608Metric, F.Cu at (177.8, 76.5)
- added J2: I2C, Connector_PinHeader_2.54mm:PinHeader_1x04_P2.54mm_Vertical, F.Cu at (124.2, 75.4)
- added J3: MOTOR, Connector_PinHeader_2.54mm:PinHeader_1x06_P2.54mm_Vertical, F.Cu at (176.0, 91.2)
- added J4: MOTOR, Connector_PinHeader_2.54mm:PinHeader_1x06_P2.54mm_Vertical, F.Cu at (124.1, 91.1)
- added R10: 100, Resistor_SMD:R_0603_1608Metric, F.Cu at (153.4, 101.6)
- added R11: 330m, Resistor_SMD:R_2512_6332Metric, F.Cu at (142.4, 110.2)
- added R12: 330m, Resistor_SMD:R_2512_6332Metric, F.Cu at (157.6, 110.2)
- added R13: 1k, Resistor_SMD:R_0603_1608Metric, F.Cu at (159.8, 101.6)
- added R14: 47k, Resistor_SMD:R_0603_1608Metric, F.Cu at (160.6, 103.9)
- added R15: 10k, Resistor_SMD:R_0603_1608Metric, F.Cu at (154.2, 103.8)
- added R16: 10k, Resistor_SMD:R_0603_1608Metric, F.Cu at (157.2, 103.9)
- added R18: 330, Resistor_SMD:R_0603_1608Metric, F.Cu at (174.7, 76.5)
- added R19: 100, Resistor_SMD:R_0603_1608Metric, F.Cu at (149.7, 80.2)
- added R20: 100, Resistor_SMD:R_0603_1608Metric, F.Cu at (127.8, 80.5)
- added R21: 100, Resistor_SMD:R_0603_1608Metric, F.Cu at (172.5, 97.3)
- added R22: 100, Resistor_SMD:R_0603_1608Metric, F.Cu at (127.6, 97.6)
- added R23: 100, Resistor_SMD:R_0603_1608Metric, F.Cu at (172.5, 98.9)
- added R24: 100, Resistor_SMD:R_0603_1608Metric, F.Cu at (127.6, 99.2)
- added R25: 100, Resistor_SMD:R_0603_1608Metric, F.Cu at (155.1, 101.6)
- added U2: STSPIN240, Package_DFN_QFN:VQFN-16-1EP_3x3mm_P0.5mm_EP1.8x1.8mm, F.Cu at (150.0, 105.1)
- added U3: LP5907MFX-3.3, Package_TO_SOT_SMD:SOT-23-5, F.Cu at (175.0, 83.7)
- added U4: HC-SR04, minimouse:HC-SR04, F.Cu at (150.0, 69.1)
- J1: value Conn_ARM_JTAG_SWD_10 -> JTAG
- moved C1 33.1 mm to (174.7, 86.4), turned to 0 degrees
- moved C5 28.6 mm to (152.3, 95.6)
- moved C6 21.4 mm to (164.9, 84.2), turned to -90 degrees
- moved C4 16.6 mm to (141.7, 86.8), turned to 180 degrees
- moved R1 12.4 mm to (161.5, 78.1), turned to 0 degrees
- moved C2 8.73 mm to (141.7, 90.8), turned to 180 degrees
- moved R6 7.38 mm to (143.7, 96.6)
- moved R7 7.34 mm to (145.3, 96.6)
- moved C3 4.98 mm to (146.3, 83.5), turned to 0 degrees
- moved R3 4.79 mm to (139.2, 96.6)
- moved R4 4.79 mm to (140.7, 96.6)
- moved R5 4.79 mm to (142.2, 96.6)
- moved R2 4.78 mm to (137.6, 96.6)
- moved J1 2.93 mm to (161.0, 83.5)
- moved R9 1.36 mm to (148.1, 80.2)
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Connections:
- R8 pad 1: /mcu/UART1_TX -> /external_uart/EXT_UART_RX
- U1 pad 43: /mcu/UART1_RX -> /external_uart/EXT_UART_TX

Commit message: TP5
Parts:
- moved R15 34.1 mm to (184.9, 89.2), turned to -90 degrees
- moved R16 31.2 mm to (182.7, 85.8), turned to -90 degrees
- moved R8 23.4 mm to (128.1, 83.2), turned to 0 degrees
- moved R11 20.6 mm to (162.2, 104.5)
- moved R12 20.2 mm to (138.2, 104.5), turned to 180 degrees
- moved R14 15.1 mm to (169.0, 91.3), turned to -90 degrees
- moved C9 11.7 mm to (165.5, 92.3)
- moved C20 8.57 mm to (119.4, 93.3), turned to 90 degrees
- moved J3 7.95 mm to (171.0, 97.4), turned to 90 degrees
- moved J4 7.93 mm to (129.6, 96.8), turned to -90 degrees
- moved C6 7.45 mm to (157.5, 83.5), turned to 180 degrees
- moved R22 7.05 mm to (122.0, 93.3), turned to -90 degrees
- moved C18 7.05 mm to (128.1, 78.1), turned to 0 degrees
- moved R6 6.95 mm to (150.6, 97.4)
- moved R7 6.95 mm to (152.2, 97.4)
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Connections:
- R21 pad 2: Net-(J3-Pin_3) -> Net-(J3-Pin_4)
- R22 pad 2: Net-(J4-Pin_3) -> Net-(J4-Pin_4)
- R23 pad 2: Net-(J3-Pin_4) -> Net-(J3-Pin_3)
- R24 pad 2: Net-(J4-Pin_4) -> Net-(J4-Pin_3)
Routing:
- net GND: track 0.00 -> 97.3 mm, vias 0 -> 27
- net +BATT: track 0.00 -> 60.3 mm, vias 0 -> 2
- net +3.3V: track 0.00 -> 26.8 mm, vias 0 -> 2
- net /mcu/TIM2_CH1: track 0.00 -> 24.2 mm
- net /motorA/MA: track 0.00 -> 22.8 mm
- net /motorB/MA: track 0.00 -> 22.4 mm
- net /mcu/TIM2_CH2: track 0.00 -> 21.5 mm
- net /mcu/BOOT0: track 0.00 -> 18.3 mm
- net Net-(U2-EN/FLT): track 0.00 -> 18.2 mm
- net Net-(U2-TOFF): track 0.00 -> 15.9 mm, vias 0 -> 3
- net /motorA/MB: track 0.00 -> 13.5 mm, vias 0 -> 2
- net /motorB/MB: track 0.00 -> 13.2 mm, vias 0 -> 2
- net /external_uart/EXT_UART_TX: track 0.00 -> 9.91 mm, vias 0 -> 2
- net /mcu/IN_B2: track 0.00 -> 9.86 mm
- net /mcu/TIM15_CH1: track 0.00 -> 9.37 mm
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- added copper zone on B.Cu, net GND
Other:
- board text added: "L.Z M1 CIM"

Commit message: LAST TP
Parts:
- removed the R7 at (152.2, 97.4)
- removed the U4 at (150.0, 69.1)
- added 3.3V_test1: TestPoint, TestPoint:TestPoint_Pad_D2.0mm, F.Cu at (123.2, 71.7)
- added 5V_TEST1: TestPoint, TestPoint:TestPoint_Pad_D2.0mm, F.Cu at (153.6, 130.8)
- added C10: 100n, Capacitor_SMD:C_0603_1608Metric, F.Cu at (136.6, 82.0)
- added D2: D_Zener, Diode_SMD:D_0402_1005Metric, F.Cu at (156.3, 133.9)
- added D3: LED, LED_SMD:LED_0603_1608Metric_Pad1.05x0.95mm_HandSolder, F.Cu at (157.9, 80.2)
- added Q1: Si2319CDS, Package_TO_SOT_SMD:SOT-23, F.Cu at (156.3, 136.5)
- added R22: 10k, Resistor_SMD:R_0603_1608Metric, F.Cu at (158.8, 134.7)
- added SW1: SW_Push, Button_Switch_SMD:SW_SPST_B3SL-1022P, F.Cu at (130.4, 84.0)
- R25: value 100 -> R
- R9: renamed from R10; value 100 -> 10k
- moved C11 57.1 mm to (122.8, 76.9)
- moved U3 49.0 mm to (126.6, 76.2), turned to 0 degrees
- moved J2 44.7 mm to (169.2, 73.6)
- moved C18 44.0 mm to (172.0, 74.7), turned to 90 degrees
- moved C12 41.8 mm to (129.6, 76.0), turned to -90 degrees
- moved D1 41.1 mm to (136.8, 74.4), turned to 90 degrees
- moved R23 39.3 mm to (135.1, 74.4), turned to 90 degrees
- moved R7 33.2 mm to (160.9, 78.3), turned to 180 degrees
- moved R17 33.1 mm to (160.9, 76.7), turned to 180 degrees
- moved C1 30.0 mm to (146.4, 81.8)
- moved R14 25.5 mm to (161.9, 100.1), turned to 0 degrees
- moved R15 24.3 mm to (161.9, 98.5), turned to 180 degrees
- moved R25 16.2 mm to (161.6, 80.2)
- moved C17 10.5 mm to (146.4, 80.2), turned to 0 degrees
- moved C8 9.77 mm to (152.8, 100.7)
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- renumbered R11 to R10, R12 to R11, R13 to R12, R14 to R13, R15 to R14, R16 to R15, R19 to R16, R20 to R17, R22 to R18, R24 to R19, R23 to R20, R18 to R23, R8 to R7, R9 to R8
Connections:
- C8 pad 1: Net-(U2-EN/FLT) -> /mcu/IN_B2
- J5 pad 2: +BATT -> Net-(J5-Pin_2)
- R18 pad 1: /mcu/TIM2_CH1 -> /mcu/TIM2_CH2
- R19 pad 1: /mcu/TIM2_CH2 -> /mcu/TIM2_CH1
- R20 pad 1: /mcu/TIM3_CH2 -> /mcu/TIM3_CH1
- R21 pad 1: /mcu/TIM3_CH1 -> /mcu/TIM3_CH2
- R25 pad 1: Net-(U2-EN/FLT) -> GND
- R25 pad 2: /mcu/IN_B2 -> Net-(D3-K)
- R9 pad 1: Net-(U2-EN/FLT) -> /mcu/IN_B2
- U1 pad 19: Net-(U1-PB1) -> /mcu/OUT_B1
- U1 pad 40: unconnected-(U1-PB4-Pad40) -> Net-(D3-A)
- U1 pad 7: /mcu/~{RESET} -> Net-(U1-NRST)
- U2 pad 13: Net-(U2-EN/FLT) -> /mcu/IN_B2
Routing:
- net +BATT: track 60.3 -> 260.0 mm, vias 2 -> 4
- net +3.3V: track 26.8 -> 89.6 mm, vias 2 -> 4
- net /mcu/TIM3_CH2: track 6.74 -> 38.5 mm
- net /motorA/MB: track 13.5 -> 43.9 mm, vias 2 -> 0
- net /motorB/MB: track 13.2 -> 42.1 mm, vias 2 -> 0
- net /mcu/TIM3_CH1: track 8.88 -> 37.4 mm
- net Net-(U1-NRST): track 0.00 -> 24.1 mm
- net /mcu/SWO: track 4.54 -> 24.8 mm, vias 2 -> 0
- net Net-(U2-EN/FLT): track 18.2 -> 0.00 mm
- net /mcu/~{RESET}: track 5.30 -> 20.5 mm, vias 2 -> 0
- net /mcu/SWDCLK: track 5.91 -> 18.9 mm, vias 2 -> 0
- net Net-(J5-Pin_2): track 0.00 -> 10.6 mm
- net Net-(U2-SENSEB): track 8.61 -> 19.0 mm
- net Net-(D3-A): track 0.00 -> 9.11 mm
- net /mcu/SWDIO: track 4.52 -> 13.1 mm, vias 2 -> 0
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Other:
- board text removed: "L.Z M1 CIM"
