File: mm_external_uart.kicad_sch (KiCad schematic)
At the start: 0 parts

Commit message: TP2
Parts:
- added C13: 0.1uF, Capacitor_SMD:C_0603_1608Metric, symbol Device:C
- added C18: 2.2uF, Capacitor_SMD:C_0603_1608Metric, symbol Device:C
- added J2: Conn_01x04, Connector_PinHeader_2.54mm:PinHeader_1x04_P2.54mm_Vertical, symbol Connector_Generic:Conn_01x04
- added R20: 100, Resistor_SMD:R_0603_1608Metric, symbol Device:R
Connections:
- new net: J2.3 (Pin_3), R20.1
- new net +BATT: C13.1, C18.1, J2.1 (Pin_1)
- new net EXT_UART_RX: J2.4 (Pin_4)
- new net EXT_UART_TX: R20.2
- new net GND: C13.2, C18.2, J2.2 (Pin_2)
Changed lines of the file:
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@@
 (kicad_sch (version 20230121) (generator eeschema)
   (paper "A4")
+  (junction (at 137.16 45.72) (diameter 0) (color 0 0 0 0)
+  )
+  (junction (at 137.16 38.1) (diameter 0) (color 0 0 0 0)
+  )
+  (wire (pts (xy 97.79 68.58) (xy 147.32 68.58))
+    (stroke (width 0) (type default))
+  )
+  (wire (pts (xy 137.16 45.72) (xy 149.86 45.72))
+    (stroke (width 0) (type default))
+  )
+  (wire (pts (xy 137.16 45.72) (xy 137.16 46.99))
+    (stroke (width 0) (type default))
+  )
+  (wire (pts (xy 137.16 36.83) (xy 137.16 38.1))
+    (stroke (width 0) (type default))
+  )
+  (wire (pts (xy 119.38 73.66) (xy 147.32 73.66))
+    (stroke (width 0) (type default))
+  )
+  (wire (pts (xy 137.16 71.12) (xy 147.32 71.12))
+    (stroke (width 0) (type default))
+  )
+  (wire (pts (xy 137.16 38.1) (xy 149.86 38.1))
+    (stroke (width 0) (type default))
+  )
+  (wire (pts (xy 119.38 71.12) (xy 129.54 71.12))
+    (stroke (width 0) (type default))
+  )
+  (wire (pts (xy 97.79 66.04) (xy 147.32 66.04))
+    (stroke (width 0) (type default))
+  )
+  (hierarchical_label "EXT_UART_RX" (shape input) (at 119.38 73.66 180) (fields_autoplaced)
+    (effects (font (size 1.27 1.27)) (justify right))
+  )
+  (hierarchical_label "EXT_UART_TX" (shape output) (at 119.38 71.12 180) (fields_autoplaced)
+    (effects (font (size 1.27 1.27)) (justify right))
+  )
+  (symbol (lib_id "power:GND") (at 97.79 68.58 0) (unit 1)
+    (in_bom yes) (on_board yes) (dnp no) (fields_autoplaced)
+    (property "Reference" "#PWR09" (at 97.79 74.93 0)
+      (effects (font (size 1.27 1.27)) hide)
+    )
+    (property "Value" "GND" (at 97.79 73.66 0)
+      (effects (font (size 1.27 1.27)))
+    )
+    (property "Footprint" "" (at 97.79 68.58 0)
+      (effects (font (size 1.27 1.27)) hide)
+    )
+    (property "Datasheet" "" (at 97.79 68.58 0)
+      (effects (font (size 1.27 1.27)) hide)
+    )
+    (pin "1")
+    (instances
+      (project "minimouse"
+        (path "/d8fa4cba-2469-4231-847f-065b6b829f44/d17bb1c7-f68a-465e-9a17-5858ef86fc30"
+          (reference "#PWR09") (unit 1)
+        )
+      )
+    )
+  )
+  (symbol (lib_id "power:GND") (at 137.16 46.99 0) (unit 1)
+    (in_bom yes) (on_board yes) (dnp no) (fields_autoplaced)
+    (property "Reference" "#PWR035" (at 137.16 53.34 0)
+      (effects (font (size 1.27 1.27)) hide)
+    )
+    (property "Value" "GND" (at 137.16 52.07 0)
+      (effects (font (size 1.27 1.27)))
+    )
+    (property "Footprint" "" (at 137.16 46.99 0)
+      (effects (font (size 1.27 1.27)) hide)
+    )
+    (property "Datasheet" "" (at 137.16 46.99 0)
+      (effects (font (size 1.27 1.27)) hide)
+    )
+    (pin "1")
+    (instances
+      (project "minimouse"
+        (path "/d8fa4cba-2469-4231-847f-065b6b829f44/d17bb1c7-f68a-465e-9a17-5858ef86fc30"
+          (reference "#PWR035") (unit 1)
+        )
+      )
+    )
+  )
+  (symbol (lib_id "Device:R") (at 133.35 71.12 270) (unit 1)
+    (in_bom yes) (on_board yes) (dnp no) (fields_autoplaced)
+    (property "Reference" "R20" (at 133.35 64.77 90)
+      (effects (font (size 1.27 1.27)) hide)
+    )
+    (property "Value" "100" (at 133.35 67.31 90)
+      (effects (font (size 1.27 1.27)))
+    )
+    (property "Footprint" "Resistor_SMD:R_0603_1608Metric" (at 133.35 69.342 90)
+      (effects (font (size 1.27 1.27)) hide)
+    )
+    (property "Datasheet" "~" (at 133.35 71.12 0)
+      (effects (font (size 1.27 1.27)) hide)
+    )
+    (pin "2")
+    (pin "1")
+    (instances
+      (project "minimouse"
+        (path "/d8fa4cba-2469-4231-847f-065b6b829f44/d17bb1c7-f68a-465e-9a17-5858ef86fc30"
+          (reference "R20") (unit 1)
+        )
+      )
+    )
+  )
+  (symbol (lib_id "Device:C") (at 137.16 41.91 0) (unit 1)
+    (in_bom yes) (on_board yes) (dnp no) (fields_autoplaced)
+    (property "Reference" "C13" (at 140.97 40.64 0)
+      (effects (font (size 1.27 1.27)) (justify left) hide)
+    )
+    (property "Value" "0.1uF" (at 140.97 43.18 0)
+      (effects (font (size 1.27 1.27)) (justify left))
+    )
+    (property "Footprint" "Capacitor_SMD:C_0603_1608Metric" (at 138.1252 45.72 0)
+      (effects (font (size 1.27 1.27)) hide)
+    )
+    (property "Datasheet" "~" (at 137.16 41.91 0)
+      (effects (font (size 1.27 1.27)) hide)
+    )
+    (pin "1")
+    (pin "2")
+    (instances
+      (project "minimouse"
+        (path "/d8fa4cba-2469-4231-847f-065b6b829f44/d17bb1c7-f68a-465e-9a17-5858ef86fc30"
+          (reference "C13") (unit 1)
+        )
+      )
+    )
+  )
+  (symbol (lib_id "power:+BATT") (at 137.16 36.83 0) (unit 1)
+    (in_bom yes) (on_board yes) (dnp no) (fields_autoplaced)
+    (property "Reference" "#PWR034" (at 137.16 40.64 0)
+      (effects (font (size 1.27 1.27)) hide)
+    )
+    (property "Value" "+BATT" (at 137.16 31.75 0)
+      (effects (font (size 1.27 1.27)))
+    )
+    (property "Footprint" "" (at 137.16 36.83 0)
+      (effects (font (size 1.27 1.27)) hide)
+    )
+    (property "Datasheet" "" (at 137.16 36.83 0)
+      (effects (font (size 1.27 1.27)) hide)
+    )
+    (pin "1")
+    (instances
+      (project "minimouse"
+        (path "/d8fa4cba-2469-4231-847f-065b6b829f44/d17bb1c7-f68a-465e-9a17-5858ef86fc30"
+          (reference "#PWR034") (unit 1)
+        )
+      )
+    )
+  )
+  (symbol (lib_id "Connector_Generic:Conn_01x04") (at 152.4 68.58 0) (unit 1)
+    (in_bom yes) (on_board yes) (dnp no) (fields_autoplaced)
+    (property "Reference" "J2" (at 154.94 68.58 0)
+      (effects (font (size 1.27 1.27)) (justify left))
+    )
+    (property "Value" "Conn_01x04" (at 154.94 71.12 0)
+      (effects (font (size 1.27 1.27)) (justify left))
+    )
+    (property "Footprint" "Connector_PinHeader_2.54mm:PinHeader_1x04_P2.54mm_Vertical" (at 152.4 68.58 0)
+      (effects (font (size 1.27 1.27)) hide)
+    )
+    (property "Datasheet" "~" (at 152.4 68.58 0)
+      (effects (font (size 1.27 1.27)) hide)
+    )
+    (pin "3")
+    (pin "2")
+    (pin "1")
+    (pin "4")
+    (instances
+      (project "minimouse"
+        (path "/d8fa4cba-2469-4231-847f-065b6b829f44/d17bb1c7-f68a-465e-9a17-5858ef86fc30"
+          (reference "J2") (unit 1)
+        )
+      )
+    )
+  )
+  (symbol (lib_id "Device:C") (at 149.86 41.91 0) (unit 1)
+    (in_bom yes) (on_board yes) (dnp no) (fields_autoplaced)
+    (property "Reference" "C18" (at 153.67 40.64 0)
+      (effects (font (size 1.27 1.27)) (justify left) hide)
+    )
+    (property "Value" "2.2uF" (at 153.67 43.18 0)
+      (effects (font (size 1.27 1.27)) (justify left))
+    )
+    (property "Footprint" "Capacitor_SMD:C_0603_1608Metric" (at 150.8252 45.72 0)
+      (effects (font (size 1.27 1.27)) hide)
+    )
+    (property "Datasheet" "~" (at 149.86 41.91 0)
+      (effects (font (size 1.27 1.27)) hide)
+    )
+    (pin "1")
+    (pin "2")
+    (instances
+      (project "minimouse"
+        (path "/d8fa4cba-2469-4231-847f-065b6b829f44/d17bb1c7-f68a-465e-9a17-5858ef86fc30"
+          (reference "C18") (unit 1)
+        )
+      )
+    )
+  )
+  (symbol (lib_id "power:+BATT") (at 97.79 66.04 0) (unit 1)
+    (in_bom yes) (on_board yes) (dnp no) (fields_autoplaced)
+    (property "Reference" "#PWR08" (at 97.79 69.85 0)
+      (effects (font (size 1.27 1.27)) hide)
+    )
+    (property "Value" "+BATT" (at 97.79 60.96 0)
+      (effects (font (size 1.27 1.27)))
+    )
+    (property "Footprint" "" (at 97.79 66.04 0)
+      (effects (font (size 1.27 1.27)) hide)
+    )
+    (property "Datasheet" "" (at 97.79 66.04 0)
+      (effects (font (size 1.27 1.27)) hide)
+    )
+    (pin "1")
+    (instances
+      (project "minimouse"
+        (path "/d8fa4cba-2469-4231-847f-065b6b829f44/d17bb1c7-f68a-465e-9a17-5858ef86fc30"
+          (reference "#PWR08") (unit 1)
+        )
+      )
+    )
+  )
 )

Commit message: TP4
Parts:
- removed C13: 0.1uF, Capacitor_SMD:C_0603_1608Metric, symbol Device:C
- J2: value Conn_01x04 -> I2C
Connections:
- net +BATT: now also J2.2 (Pin_2); no longer J2.1 (Pin_1)
- net GND: now also J2.1 (Pin_1); no longer J2.2 (Pin_2)
Changed lines of the file:
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@@
 (kicad_sch (version 20230121) (generator eeschema)
   (paper "A4")
-  (junction (at 137.16 45.72) (diameter 0) (color 0 0 0 0)
-  )
-  (junction (at 137.16 38.1) (diameter 0) (color 0 0 0 0)
-  )
   (wire (pts (xy 97.79 68.58) (xy 147.32 68.58))
-    (stroke (width 0) (type default))
-  )
-  (wire (pts (xy 137.16 45.72) (xy 149.86 45.72))
     (stroke (width 0) (type default))
   )
@@
     (stroke (width 0) (type default))
   )
-  (wire (pts (xy 137.16 36.83) (xy 137.16 38.1))
+  (wire (pts (xy 137.16 38.1) (xy 137.16 36.83))
     (stroke (width 0) (type default))
   )
@@
     (stroke (width 0) (type default))
   )
-  (wire (pts (xy 137.16 38.1) (xy 149.86 38.1))
-    (stroke (width 0) (type default))
-  )
   (wire (pts (xy 119.38 71.12) (xy 129.54 71.12))
     (stroke (width 0) (type default))
   )
-  (wire (pts (xy 97.79 66.04) (xy 147.32 66.04))
+  (wire (pts (xy 87.63 66.04) (xy 87.63 72.39))
+    (stroke (width 0) (type default))
+  )
+  (wire (pts (xy 87.63 66.04) (xy 147.32 66.04))
+    (stroke (width 0) (type default))
+  )
+  (wire (pts (xy 97.79 60.96) (xy 97.79 68.58))
     (stroke (width 0) (type default))
   )
@@
   (hierarchical_label "EXT_UART_TX" (shape output) (at 119.38 71.12 180) (fields_autoplaced)
     (effects (font (size 1.27 1.27)) (justify right))
-  )
-  (symbol (lib_id "power:GND") (at 97.79 68.58 0) (unit 1)
-    (in_bom yes) (on_board yes) (dnp no) (fields_autoplaced)
-    (property "Reference" "#PWR09" (at 97.79 74.93 0)
-      (effects (font (size 1.27 1.27)) hide)
-    )
-    (property "Value" "GND" (at 97.79 73.66 0)
-      (effects (font (size 1.27 1.27)))
-    )
-    (property "Footprint" "" (at 97.79 68.58 0)
-      (effects (font (size 1.27 1.27)) hide)
-    )
-    (property "Datasheet" "" (at 97.79 68.58 0)
-      (effects (font (size 1.27 1.27)) hide)
-    )
-    (pin "1")
-    (instances
-      (project "minimouse"
-        (path "/d8fa4cba-2469-4231-847f-065b6b829f44/d17bb1c7-f68a-465e-9a17-5858ef86fc30"
-          (reference "#PWR09") (unit 1)
-        )
-      )
-    )
   )
   (symbol (lib_id "power:GND") (at 137.16 46.99 0) (unit 1)
@@
     )
   )
-  (symbol (lib_id "Device:C") (at 137.16 41.91 0) (unit 1)
-    (in_bom yes) (on_board yes) (dnp no) (fields_autoplaced)
-    (property "Reference" "C13" (at 140.97 40.64 0)
-      (effects (font (size 1.27 1.27)) (justify left) hide)
-    )
-    (property "Value" "0.1uF" (at 140.97 43.18 0)
-      (effects (font (size 1.27 1.27)) (justify left))
-    )
-    (property "Footprint" "Capacitor_SMD:C_0603_1608Metric" (at 138.1252 45.72 0)
-      (effects (font (size 1.27 1.27)) hide)
-    )
-    (property "Datasheet" "~" (at 137.16 41.91 0)
-      (effects (font (size 1.27 1.27)) hide)
-    )
-    (pin "1")
-    (pin "2")
-    (instances
-      (project "minimouse"
-        (path "/d8fa4cba-2469-4231-847f-065b6b829f44/d17bb1c7-f68a-465e-9a17-5858ef86fc30"
-          (reference "C13") (unit 1)
-        )
-      )
-    )
-  )
   (symbol (lib_id "power:+BATT") (at 137.16 36.83 0) (unit 1)
     (in_bom yes) (on_board yes) (dnp no) (fields_autoplaced)
@@
       (effects (font (size 1.27 1.27)) (justify left))
     )
-    (property "Value" "Conn_01x04" (at 154.94 71.12 0)
+    (property "Value" "I2C" (at 154.94 71.12 0)
       (effects (font (size 1.27 1.27)) (justify left))
     )
@@
     )
   )
-  (symbol (lib_id "Device:C") (at 149.86 41.91 0) (unit 1)
+  (symbol (lib_id "Device:C") (at 137.16 41.91 0) (unit 1)
     (in_bom yes) (on_board yes) (dnp no) (fields_autoplaced)
-    (property "Reference" "C18" (at 153.67 40.64 0)
+    (property "Reference" "C18" (at 140.97 40.64 0)
       (effects (font (size 1.27 1.27)) (justify left) hide)
     )
-    (property "Value" "2.2uF" (at 153.67 43.18 0)
+    (property "Value" "2.2uF" (at 140.97 43.18 0)
       (effects (font (size 1.27 1.27)) (justify left))
     )
-    (property "Footprint" "Capacitor_SMD:C_0603_1608Metric" (at 150.8252 45.72 0)
+    (property "Footprint" "Capacitor_SMD:C_0603_1608Metric" (at 138.1252 45.72 0)
       (effects (font (size 1.27 1.27)) hide)
     )
-    (property "Datasheet" "~" (at 149.86 41.91 0)
+    (property "Datasheet" "~" (at 137.16 41.91 0)
       (effects (font (size 1.27 1.27)) hide)
     )
@@
     )
   )
-  (symbol (lib_id "power:+BATT") (at 97.79 66.04 0) (unit 1)
+  (symbol (lib_id "power:+BATT") (at 97.79 60.96 0) (unit 1)
     (in_bom yes) (on_board yes) (dnp no) (fields_autoplaced)
-    (property "Reference" "#PWR08" (at 97.79 69.85 0)
+    (property "Reference" "#PWR09" (at 97.79 64.77 0)
       (effects (font (size 1.27 1.27)) hide)
     )
-    (property "Value" "+BATT" (at 97.79 60.96 0)
+    (property "Value" "+BATT" (at 97.79 55.88 0)
       (effects (font (size 1.27 1.27)))
     )
-    (property "Footprint" "" (at 97.79 66.04 0)
+    (property "Footprint" "" (at 97.79 60.96 0)
       (effects (font (size 1.27 1.27)) hide)
     )
-    (property "Datasheet" "" (at 97.79 66.04 0)
+    (property "Datasheet" "" (at 97.79 60.96 0)
       (effects (font (size 1.27 1.27)) hide)
     )
+    (pin "1")
+    (instances
+      (project "minimouse"
+        (path "/d8fa4cba-2469-4231-847f-065b6b829f44/d17bb1c7-f68a-465e-9a17-5858ef86fc30"
+          (reference "#PWR09") (unit 1)
+        )
+      )
+    )
+  )
+  (symbol (lib_id "power:GND") (at 87.63 72.39 0) (unit 1)
+    (in_bom yes) (on_board yes) (dnp no) (fields_autoplaced)
+    (property "Reference" "#PWR08" (at 87.63 78.74 0)
+      (effects (font (size 1.27 1.27)) hide)
+    )
+    (property "Value" "GND" (at 87.63 77.47 0)
+      (effects (font (size 1.27 1.27)))
+    )
+    (property "Footprint" "" (at 87.63 72.39 0)
+      (effects (font (size 1.27 1.27)) hide)
+    )
+    (property "Datasheet" "" (at 87.63 72.39 0)
+      (effects (font (size 1.27 1.27)) hide)
+    )

Commit message: LAST TP
Parts:
- renumbered R20 to R17
Changed lines of the file:
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@@
   (symbol (lib_id "Device:R") (at 133.35 71.12 270) (unit 1)
     (in_bom yes) (on_board yes) (dnp no) (fields_autoplaced)
-    (property "Reference" "R20" (at 133.35 64.77 90)
+    (property "Reference" "R17" (at 133.35 64.77 90)
       (effects (font (size 1.27 1.27)) hide)
     )
@@
       (project "minimouse"
         (path "/d8fa4cba-2469-4231-847f-065b6b829f44/d17bb1c7-f68a-465e-9a17-5858ef86fc30"
-          (reference "R20") (unit 1)
+          (reference "R17") (unit 1)
         )
       )
