File: mm_mcu.kicad_sch (KiCad schematic)
At the start: 18 parts, among them J1 Conn_ARM_JTAG_SWD_10, U1 STM32F030C8Tx

Commit message: TP4
Parts:
- J1: value Conn_ARM_JTAG_SWD_10 -> JTAG
Changed lines of the file:
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@@
       (effects (font (size 1.27 1.27)) (justify right))
     )
-    (property "Value" "Conn_ARM_JTAG_SWD_10" (at 38.1 165.1 0)
+    (property "Value" "JTAG" (at 38.1 165.1 0)
       (effects (font (size 1.27 1.27)) (justify right))
     )

Commit message: LAST TP
Parts:
- removed R7: 100, Resistor_SMD:R_0603_1608Metric, symbol Device:R
- added C10: 100n, Capacitor_SMD:C_0603_1608Metric, symbol Device:C
- added D3: LED, LED_SMD:LED_0603_1608Metric_Pad1.05x0.95mm_HandSolder, symbol Device:LED
- added R25: R, Resistor_SMD:R_0603_1608Metric, symbol Device:R
- added SW1: SW_Push, Button_Switch_SMD:SW_SPST_B3SL-1022P, symbol Switch:SW_Push
- renumbered R8 to R7, R9 to R8
Connections:
- net GND: now also C10.1, R25.1, SW1.1
- net OUT_B1: now also U1.19 (PB1)
- net ~{RESET}: no longer U1.7 (NRST)
- net at U1.40 (PB4): now also D3.2 (A)
- new net: C10.2, SW1.2, U1.7 (NRST)
- new net: D3.1 (K), R25.2
- no-connect marks 22 -> 21
