File: mm_motor.kicad_sch (KiCad schematic)
At the start: 1 part, among them M1 N20_encoder

Commit message: TP2
Parts:
- added C13: 0.1uF, Capacitor_SMD:C_0603_1608Metric, symbol Device:C
- added C13: 2.2uF, Capacitor_SMD:C_0603_1608Metric, symbol Device:C
- added J3: Conn_01x06, Connector_PinHeader_2.54mm:PinHeader_1x06_P2.54mm_Vertical, symbol Connector_Generic:Conn_01x06
- added R22, R24: 100, Resistor_SMD:R_0603_1608Metric, symbol Device:R
Connections:
- net C1: now also R22.1
- net C2: now also R24.1
- net MA: now also J3.1 (Pin_1)
- net MB: now also J3.6 (Pin_6)
- new net: J3.3 (Pin_3), R22.2
- new net: J3.4 (Pin_4), R24.2
- new net +BATT: C13.1, C13.1, J3.5 (Pin_5)
- new net GND: C13.2, C13.2, J3.2 (Pin_2)
Other:
- moved on the sheet: M1

Commit message: TP4
Parts:
- removed C13: 0.1uF, Capacitor_SMD:C_0603_1608Metric, symbol Device:C
- J3: value Conn_01x06 -> MOTOR
- renumbered C13 to C19
Changed lines of the file:
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@@
 (kicad_sch (version 20230121) (generator eeschema)
   (paper "A4")
-  (junction (at 101.6 67.31) (diameter 0) (color 0 0 0 0)
-  )
-  (junction (at 101.6 74.93) (diameter 0) (color 0 0 0 0)
-  )
   (wire (pts (xy 129.54 91.44) (xy 133.35 91.44))
     (stroke (width 0) (type default))
@@
     (stroke (width 0) (type default))
   )
-  (wire (pts (xy 101.6 66.04) (xy 101.6 67.31))
-    (stroke (width 0) (type default))
-  )
-  (wire (pts (xy 101.6 67.31) (xy 114.3 67.31))
-    (stroke (width 0) (type default))
-  )
-  (wire (pts (xy 101.6 74.93) (xy 114.3 74.93))
+  (wire (pts (xy 101.6 67.31) (xy 101.6 66.04))
     (stroke (width 0) (type default))
   )
@@
   (symbol (lib_id "power:+BATT") (at 101.6 66.04 0) (unit 1)
     (in_bom yes) (on_board yes) (dnp no) (fields_autoplaced)
-    (property "Reference" "#PWR035" (at 101.6 69.85 0)
+    (property "Reference" "#PWR040" (at 101.6 69.85 0)
       (effects (font (size 1.27 1.27)) hide)
     )
@@
     (instances
       (project "minimouse"
-        (path "/d8fa4cba-2469-4231-847f-065b6b829f44/d17bb1c7-f68a-465e-9a17-5858ef86fc30"
-          (reference "#PWR035") (unit 1)
-        )
         (path "/d8fa4cba-2469-4231-847f-065b6b829f44/7f113667-692a-4f4d-b16f-621d32f3f136"
           (reference "#PWR040") (unit 1)
@@
   (symbol (lib_id "power:GND") (at 101.6 76.2 0) (unit 1)
     (in_bom yes) (on_board yes) (dnp no) (fields_autoplaced)
-    (property "Reference" "#PWR034" (at 101.6 82.55 0)
+    (property "Reference" "#PWR041" (at 101.6 82.55 0)
       (effects (font (size 1.27 1.27)) hide)
     )
@@
     (instances
       (project "minimouse"
-        (path "/d8fa4cba-2469-4231-847f-065b6b829f44/d17bb1c7-f68a-465e-9a17-5858ef86fc30"
-          (reference "#PWR034") (unit 1)
-        )
         (path "/d8fa4cba-2469-4231-847f-065b6b829f44/7f113667-692a-4f4d-b16f-621d32f3f136"
           (reference "#PWR041") (unit 1)
@@
       (effects (font (size 1.27 1.27)) (justify left))
     )
-    (property "Value" "Conn_01x06" (at 140.97 93.98 0)
+    (property "Value" "MOTOR" (at 140.97 93.98 0)
       (effects (font (size 1.27 1.27)) (justify left))
     )
@@
   (symbol (lib_id "Device:C") (at 101.6 71.12 0) (unit 1)
     (in_bom yes) (on_board yes) (dnp no) (fields_autoplaced)
-    (property "Reference" "C13" (at 105.41 69.85 0)
+    (property "Reference" "C19" (at 105.41 69.85 0)
       (effects (font (size 1.27 1.27)) (justify left) hide)
     )
-    (property "Value" "0.1uF" (at 105.41 72.39 0)
+    (property "Value" "2.2uF" (at 105.41 72.39 0)
       (effects (font (size 1.27 1.27)) (justify left))
     )
@@
     (instances
       (project "minimouse"
-        (path "/d8fa4cba-2469-4231-847f-065b6b829f44/d17bb1c7-f68a-465e-9a17-5858ef86fc30"
-          (reference "C13") (unit 1)
-        )
-        (path "/d8fa4cba-2469-4231-847f-065b6b829f44/7f113667-692a-4f4d-b16f-621d32f3f136"
-          (reference "C15") (unit 1)
-        )
-        (path "/d8fa4cba-2469-4231-847f-065b6b829f44/3975acd0-18ad-47bc-9ce1-d8c4d864aafe"
-          (reference "C16") (unit 1)
-        )
-      )
-    )
-  )
-  (symbol (lib_id "Device:C") (at 114.3 71.12 0) (unit 1)
-    (in_bom yes) (on_board yes) (dnp no) (fields_autoplaced)
-    (property "Reference" "C13" (at 118.11 69.85 0)
-      (effects (font (size 1.27 1.27)) (justify left) hide)
-    )
-    (property "Value" "2.2uF" (at 118.11 72.39 0)
-      (effects (font (size 1.27 1.27)) (justify left))
-    )
-    (property "Footprint" "Capacitor_SMD:C_0603_1608Metric" (at 115.2652 74.93 0)
-      (effects (font (size 1.27 1.27)) hide)
-    )
-    (property "Datasheet" "~" (at 114.3 71.12 0)
-      (effects (font (size 1.27 1.27)) hide)
-    )
-    (pin "1")
-    (pin "2")
-    (instances
-      (project "minimouse"
-        (path "/d8fa4cba-2469-4231-847f-065b6b829f44/d17bb1c7-f68a-465e-9a17-5858ef86fc30"
-          (reference "C13") (unit 1)
-        )
         (path "/d8fa4cba-2469-4231-847f-065b6b829f44/7f113667-692a-4f4d-b16f-621d32f3f136"
           (reference "C19") (unit 1)

Commit message: TP5
Connections:
- net at R22.2: now also J3.4 (Pin_4); no longer J3.3 (Pin_3)
- net at R24.2: now also J3.3 (Pin_3); no longer J3.4 (Pin_4)
Changed lines of the file:
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@@
 (kicad_sch (version 20230121) (generator eeschema)
   (paper "A4")
+  (wire (pts (xy 118.11 91.44) (xy 121.92 91.44))
+    (stroke (width 0) (type default))
+  )
+  (wire (pts (xy 118.11 86.36) (xy 133.35 86.36))
+    (stroke (width 0) (type default))
+  )
+  (wire (pts (xy 101.6 74.93) (xy 101.6 76.2))
+    (stroke (width 0) (type default))
+  )
+  (wire (pts (xy 118.11 93.98) (xy 121.92 93.98))
+    (stroke (width 0) (type default))
+  )
+  (wire (pts (xy 87.63 90.17) (xy 87.63 88.9))
+    (stroke (width 0) (type default))
+  )
+  (wire (pts (xy 129.54 93.98) (xy 133.35 93.98))
+    (stroke (width 0) (type default))
+  )
+  (wire (pts (xy 101.6 67.31) (xy 101.6 66.04))
+    (stroke (width 0) (type default))
+  )
+  (wire (pts (xy 87.63 88.9) (xy 133.35 88.9))
+    (stroke (width 0) (type default))
+  )
+  (wire (pts (xy 101.6 96.52) (xy 133.35 96.52))
+    (stroke (width 0) (type default))
+  )
+  (wire (pts (xy 118.11 99.06) (xy 133.35 99.06))
+    (stroke (width 0) (type default))
+  )
   (wire (pts (xy 129.54 91.44) (xy 133.35 91.44))
     (stroke (width 0) (type default))
   )
-  (wire (pts (xy 118.11 86.36) (xy 133.35 86.36))
-    (stroke (width 0) (type default))
-  )
-  (wire (pts (xy 101.6 74.93) (xy 101.6 76.2))
-    (stroke (width 0) (type default))
-  )
-  (wire (pts (xy 118.11 93.98) (xy 121.92 93.98))
-    (stroke (width 0) (type default))
-  )
-  (wire (pts (xy 118.11 91.44) (xy 121.92 91.44))
-    (stroke (width 0) (type default))
-  )
-  (wire (pts (xy 87.63 90.17) (xy 87.63 88.9))
-    (stroke (width 0) (type default))
-  )
-  (wire (pts (xy 101.6 67.31) (xy 101.6 66.04))
-    (stroke (width 0) (type default))
-  )
-  (wire (pts (xy 87.63 88.9) (xy 133.35 88.9))
-    (stroke (width 0) (type default))
-  )
-  (wire (pts (xy 101.6 96.52) (xy 133.35 96.52))
-    (stroke (width 0) (type default))
-  )
-  (wire (pts (xy 118.11 99.06) (xy 133.35 99.06))
-    (stroke (width 0) (type default))
-  )
-  (wire (pts (xy 129.54 93.98) (xy 133.35 93.98))
-    (stroke (width 0) (type default))
-  )
-  (hierarchical_label "C1" (shape output) (at 118.11 91.44 180) (fields_autoplaced)
-    (effects (font (size 1.27 1.27)) (justify right))
-  )
-  (hierarchical_label "C2" (shape output) (at 118.11 93.98 180) (fields_autoplaced)
+  (hierarchical_label "C1" (shape output) (at 118.11 93.98 180) (fields_autoplaced)
+    (effects (font (size 1.27 1.27)) (justify right))
+  )
+  (hierarchical_label "C2" (shape output) (at 118.11 91.44 180) (fields_autoplaced)
     (effects (font (size 1.27 1.27)) (justify right))
   )
@@
     )
   )
-  (symbol (lib_id "Device:R") (at 125.73 91.44 90) (unit 1)
-    (in_bom yes) (on_board yes) (dnp no) (fields_autoplaced)
-    (property "Reference" "R22" (at 125.73 85.09 90)
-      (effects (font (size 1.27 1.27)) hide)
-    )
-    (property "Value" "100" (at 125.73 87.63 90)
-      (effects (font (size 1.27 1.27)) hide)
-    )
-    (property "Footprint" "Resistor_SMD:R_0603_1608Metric" (at 125.73 93.218 90)
-      (effects (font (size 1.27 1.27)) hide)
-    )
-    (property "Datasheet" "~" (at 125.73 91.44 0)
+  (symbol (lib_id "Device:R") (at 125.73 93.98 90) (unit 1)
+    (in_bom yes) (on_board yes) (dnp no) (fields_autoplaced)
+    (property "Reference" "R22" (at 125.73 87.63 90)
+      (effects (font (size 1.27 1.27)) hide)
+    )
+    (property "Value" "100" (at 125.73 90.17 90)
+      (effects (font (size 1.27 1.27)) hide)
+    )
+    (property "Footprint" "Resistor_SMD:R_0603_1608Metric" (at 125.73 95.758 90)
+      (effects (font (size 1.27 1.27)) hide)
+    )
+    (property "Datasheet" "~" (at 125.73 93.98 0)
       (effects (font (size 1.27 1.27)) hide)
     )
@@
     )
   )
-  (symbol (lib_id "Device:R") (at 125.73 93.98 90) (unit 1)
-    (in_bom yes) (on_board yes) (dnp no) (fields_autoplaced)
-    (property "Reference" "R24" (at 125.73 87.63 90)
-      (effects (font (size 1.27 1.27)) hide)
-    )
-    (property "Value" "100" (at 125.73 90.17 90)
-      (effects (font (size 1.27 1.27)) hide)
-    )
-    (property "Footprint" "Resistor_SMD:R_0603_1608Metric" (at 125.73 95.758 90)
-      (effects (font (size 1.27 1.27)) hide)
-    )
-    (property "Datasheet" "~" (at 125.73 93.98 0)
-      (effects (font (size 1.27 1.27)) hide)
-    )
+  (symbol (lib_id "Device:R") (at 125.73 91.44 90) (unit 1)
+    (in_bom yes) (on_board yes) (dnp no) (fields_autoplaced)
+    (property "Reference" "R24" (at 125.73 85.09 90)
+      (effects (font (size 1.27 1.27)) hide)
+    )
+    (property "Value" "100" (at 125.73 87.63 90)
+      (effects (font (size 1.27 1.27)) hide)
+    )
+    (property "Footprint" "Resistor_SMD:R_0603_1608Metric" (at 125.73 93.218 90)
+      (effects (font (size 1.27 1.27)) hide)
+    )
+    (property "Datasheet" "~" (at 125.73 91.44 0)
+      (effects (font (size 1.27 1.27)) hide)
+    )

Commit message: LAST TP
Parts:
- renumbered R22 to R18, R24 to R19
Connections:
- net C1: now also R19.1; no longer R18.1
- net C2: now also R18.1; no longer R19.1
Changed lines of the file:
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@@
 (kicad_sch (version 20230121) (generator eeschema)
   (paper "A4")
+  (wire (pts (xy 118.11 86.36) (xy 133.35 86.36))
+    (stroke (width 0) (type default))
+  )
+  (wire (pts (xy 101.6 74.93) (xy 101.6 76.2))
+    (stroke (width 0) (type default))
+  )
+  (wire (pts (xy 87.63 90.17) (xy 87.63 88.9))
+    (stroke (width 0) (type default))
+  )
+  (wire (pts (xy 129.54 93.98) (xy 133.35 93.98))
+    (stroke (width 0) (type default))
+  )
+  (wire (pts (xy 101.6 67.31) (xy 101.6 66.04))
+    (stroke (width 0) (type default))
+  )
+  (wire (pts (xy 87.63 88.9) (xy 133.35 88.9))
+    (stroke (width 0) (type default))
+  )
+  (wire (pts (xy 101.6 96.52) (xy 133.35 96.52))
+    (stroke (width 0) (type default))
+  )
   (wire (pts (xy 118.11 91.44) (xy 121.92 91.44))
     (stroke (width 0) (type default))
   )
-  (wire (pts (xy 118.11 86.36) (xy 133.35 86.36))
-    (stroke (width 0) (type default))
-  )
-  (wire (pts (xy 101.6 74.93) (xy 101.6 76.2))
+  (wire (pts (xy 118.11 99.06) (xy 133.35 99.06))
+    (stroke (width 0) (type default))
+  )
+  (wire (pts (xy 129.54 91.44) (xy 133.35 91.44))
     (stroke (width 0) (type default))
   )
@@
     (stroke (width 0) (type default))
   )
-  (wire (pts (xy 87.63 90.17) (xy 87.63 88.9))
-    (stroke (width 0) (type default))
-  )
-  (wire (pts (xy 129.54 93.98) (xy 133.35 93.98))
-    (stroke (width 0) (type default))
-  )
-  (wire (pts (xy 101.6 67.31) (xy 101.6 66.04))
-    (stroke (width 0) (type default))
-  )
-  (wire (pts (xy 87.63 88.9) (xy 133.35 88.9))
-    (stroke (width 0) (type default))
-  )
-  (wire (pts (xy 101.6 96.52) (xy 133.35 96.52))
-    (stroke (width 0) (type default))
-  )
-  (wire (pts (xy 118.11 99.06) (xy 133.35 99.06))
-    (stroke (width 0) (type default))
-  )
-  (wire (pts (xy 129.54 91.44) (xy 133.35 91.44))
-    (stroke (width 0) (type default))
-  )
-  (hierarchical_label "C1" (shape output) (at 118.11 93.98 180) (fields_autoplaced)
-    (effects (font (size 1.27 1.27)) (justify right))
-  )
-  (hierarchical_label "C2" (shape output) (at 118.11 91.44 180) (fields_autoplaced)
+  (hierarchical_label "C1" (shape output) (at 118.11 91.44 180) (fields_autoplaced)
+    (effects (font (size 1.27 1.27)) (justify right))
+  )
+  (hierarchical_label "C2" (shape output) (at 118.11 93.98 180) (fields_autoplaced)
     (effects (font (size 1.27 1.27)) (justify right))
   )
@@
   (symbol (lib_id "Device:R") (at 125.73 93.98 90) (unit 1)
     (in_bom yes) (on_board yes) (dnp no) (fields_autoplaced)
-    (property "Reference" "R22" (at 125.73 87.63 90)
+    (property "Reference" "R18" (at 125.73 87.63 90)
       (effects (font (size 1.27 1.27)) hide)
     )
@@
       (project "minimouse"
         (path "/d8fa4cba-2469-4231-847f-065b6b829f44/3975acd0-18ad-47bc-9ce1-d8c4d864aafe"
-          (reference "R22") (unit 1)
+          (reference "R18") (unit 1)
         )
         (path "/d8fa4cba-2469-4231-847f-065b6b829f44/7f113667-692a-4f4d-b16f-621d32f3f136"
@@
   (symbol (lib_id "Device:R") (at 125.73 91.44 90) (unit 1)
     (in_bom yes) (on_board yes) (dnp no) (fields_autoplaced)
-    (property "Reference" "R24" (at 125.73 85.09 90)
+    (property "Reference" "R19" (at 125.73 85.09 90)
       (effects (font (size 1.27 1.27)) hide)
     )
@@
       (project "minimouse"
         (path "/d8fa4cba-2469-4231-847f-065b6b829f44/3975acd0-18ad-47bc-9ce1-d8c4d864aafe"
-          (reference "R24") (unit 1)
-        )
-        (path "/d8fa4cba-2469-4231-847f-065b6b829f44/7f113667-692a-4f4d-b16f-621d32f3f136"
-          (reference "R23") (unit 1)
-        )
-      )
+          (reference "R19") (unit 1)
+        )
+        (path "/d8fa4cba-2469-4231-847f-065b6b829f44/7f113667-692a-4f4d-b16f-621d32f3f136"
+          (reference "R20") (unit 1)
+        )
+      )
