File: mm_motor_control.kicad_sch (KiCad schematic)
At the start: 0 parts

Commit message: TP2
Parts:
- added C10: 1nF, Capacitor_SMD:C_0603_1608Metric, symbol Device:C
- added C7: 2.2uF, Capacitor_SMD:C_0603_1608Metric, symbol Device:C
- added C8: 0.1uF, Capacitor_SMD:C_0603_1608Metric, symbol Device:C
- added C9: 22nF, Capacitor_SMD:C_0603_1608Metric, symbol Device:C
- added R10: 100, symbol Device:R
- added R11, R12: 330m, Resistor_SMD:R_0603_1608Metric, symbol Device:R
- added R13: 1.3k, Resistor_SMD:R_0603_1608Metric, symbol Device:R
- added R14: 47k, Resistor_SMD:R_0603_1608Metric, symbol Device:R
- added R15, R16: 10k, Resistor_SMD:R_0603_1608Metric, symbol Device:R
- added R17: 330, Resistor_SMD:R_0603_1608Metric, symbol Device:R
- added R20: 100, Resistor_SMD:R_0603_1608Metric, symbol Device:R
- added U2: STSPIN240, Package_DFN_QFN:VQFN-16-1EP_3x3mm_P0.5mm_EP1.8x1.8mm, symbol Driver_Motor:STSPIN240
Connections:
- net EN: now also R10.2
- net FAULT: now also R20.2
- net OUT_A1: now also U2.3 (OUTA1)
- net OUT_A2: now also U2.5 (OUTA2)
- net OUT_B1: now also U2.10 (OUTB1)
- net OUT_B2: now also U2.8 (OUTB2)
- net PHASE_A: now also U2.1 (PHA)
- net PHASE_B: now also U2.15 (PHB)
- net PWM_A: now also U2.2 (PWMA)
- net PWM_B: now also U2.16 (PWMB)
- net STBY/RESET: now also C10.1, R17.2, U2.14 (STBY/RESET)
- new net: R13.1, R14.1, U2.12 (TOFF)
- new net: C9.1, R13.2
- new net: C8.1, R10.1, R20.1, U2.13 (EN/FLT)
- new net: R12.1, U2.4 (SENSEA)
- new net: R11.1, U2.9 (SENSEB)
- new net +3.3V: R17.1
- new net +BATT: C7.1, R16.1, U2.6 (VS)
- new net GND: C10.2, C7.2, C8.2, C9.2, R11.2, R12.2, R14.2, R15.2, U2.17 (EPAD), U2.7 (GND)
- new net REF: R15.1, R16.2, U2.11 (REF)

Commit message: TP4
Parts:
- removed C10: 1nF, Capacitor_SMD:C_0603_1608Metric, symbol Device:C
- removed R17: 330, Resistor_SMD:R_0603_1608Metric, symbol Device:R
- R10: footprint (none) -> Resistor_SMD:R_0603_1608Metric
- R11, R12: footprint Resistor_SMD:R_0603_1608Metric -> Resistor_SMD:R_2512_6332Metric
- R13: value 1.3k -> 1k
- renumbered R20 to R25
Changed lines of the file:
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@@
   (junction (at 124.46 104.14) (diameter 0) (color 0 0 0 0)
   )
-  (junction (at 64.77 125.73) (diameter 0) (color 0 0 0 0)
-  )
   (junction (at 113.03 133.35) (diameter 0) (color 0 0 0 0)
   )
@@
     (stroke (width 0) (type default))
   )
-  (wire (pts (xy 111.76 96.52) (xy 137.16 96.52))
+  (wire (pts (xy 107.95 96.52) (xy 137.16 96.52))
     (stroke (width 0) (type default))
   )
@@
     (stroke (width 0) (type default))
   )
-  (wire (pts (xy 64.77 110.49) (xy 64.77 115.57))
-    (stroke (width 0) (type default))
-  )
   (wire (pts (xy 88.9 107.95) (xy 88.9 111.76))
     (stroke (width 0) (type default))
@@
     (stroke (width 0) (type default))
   )
-  (wire (pts (xy 64.77 125.73) (xy 72.39 125.73))
-    (stroke (width 0) (type default))
-  )
   (wire (pts (xy 149.86 109.22) (xy 149.86 111.76))
     (stroke (width 0) (type default))
   )
-  (wire (pts (xy 64.77 135.89) (xy 64.77 139.7))
-    (stroke (width 0) (type default))
-  )
   (wire (pts (xy 165.1 91.44) (xy 198.12 91.44))
     (stroke (width 0) (type default))
@@
     (stroke (width 0) (type default))
   )
-  (wire (pts (xy 64.77 123.19) (xy 64.77 125.73))
-    (stroke (width 0) (type default))
-  )
   (wire (pts (xy 176.53 83.82) (xy 180.34 83.82))
     (stroke (width 0) (type default))
@@
     (stroke (width 0) (type default))
   )
-  (wire (pts (xy 64.77 125.73) (xy 64.77 128.27))
-    (stroke (width 0) (type default))
-  )
   (wire (pts (xy 149.86 52.07) (xy 149.86 55.88))
     (stroke (width 0) (type default))
@@
     (stroke (width 0) (type default))
   )
-  (wire (pts (xy 55.88 125.73) (xy 64.77 125.73))
-    (stroke (width 0) (type default))
-  )
   (wire (pts (xy 88.9 93.98) (xy 88.9 100.33))
     (stroke (width 0) (type default))
@@
   (wire (pts (xy 165.1 96.52) (xy 168.91 96.52))
     (stroke (width 0) (type default))
-  )
-  (label "STBY" (at 111.76 96.52 0) (fields_autoplaced)
-    (effects (font (size 1.27 1.27)) (justify left bottom))
-  )
-  (label "STBY" (at 72.39 125.73 0) (fields_autoplaced)
-    (effects (font (size 1.27 1.27)) (justify left bottom))
   )
   (label "REF" (at 127 101.6 0) (fields_autoplaced)
@@
     (effects (font (size 1.27 1.27)) (justify left))
   )
+  (hierarchical_label "STBY{slash}RESET" (shape input) (at 107.95 96.52 180) (fields_autoplaced)
+    (effects (font (size 1.27 1.27)) (justify right))
+  )
   (hierarchical_label "OUT_B1" (shape passive) (at 198.12 91.44 0) (fields_autoplaced)
     (effects (font (size 1.27 1.27)) (justify left))
   )
-  (hierarchical_label "STBY{slash}RESET" (shape input) (at 55.88 125.73 180) (fields_autoplaced)
-    (effects (font (size 1.27 1.27)) (justify right))
-  )
   (hierarchical_label "EN" (shape input) (at 69.85 93.98 180) (fields_autoplaced)
     (effects (font (size 1.27 1.27)) (justify right))
   )
-  (symbol (lib_id "Device:R") (at 64.77 119.38 0) (unit 1)
-    (in_bom yes) (on_board yes) (dnp no) (fields_autoplaced)
-    (property "Reference" "R17" (at 58.42 119.38 90)
-      (effects (font (size 1.27 1.27)) hide)
-    )
-    (property "Value" "330" (at 67.31 119.38 0)
-      (effects (font (size 1.27 1.27)) (justify left))
-    )
-    (property "Footprint" "Resistor_SMD:R_0603_1608Metric" (at 62.992 119.38 90)
-      (effects (font (size 1.27 1.27)) hide)
-    )
-    (property "Datasheet" "~" (at 64.77 119.38 0)
-      (effects (font (size 1.27 1.27)) hide)
-    )
-    (pin "1")
-    (pin "2")
-    (instances
-      (project "minimouse"
-        (path "/d8fa4cba-2469-4231-847f-065b6b829f44/0999fad3-9a14-4ede-b729-a71c3dbbdf8e"
-          (reference "R17") (unit 1)
-        )
-      )
-    )
-  )
   (symbol (lib_id "Device:R") (at 113.03 114.3 0) (unit 1)
     (in_bom yes) (on_board yes) (dnp no) (fields_autoplaced)
@@
       (effects (font (size 1.27 1.27)) (justify left) hide)
     )
-    (property "Value" "1.3k" (at 115.57 115.57 0)
+    (property "Value" "1k" (at 115.57 115.57 0)
       (effects (font (size 1.27 1.27)) (justify left))
     )
@@
     )
   )
-  (symbol (lib_id "Device:C") (at 64.77 132.08 0) (unit 1)
-    (in_bom yes) (on_board yes) (dnp no) (fields_autoplaced)
-    (property "Reference" "C10" (at 68.58 130.81 0)
-      (effects (font (size 1.27 1.27)) (justify left) hide)
-    )
-    (property "Value" "1nF" (at 68.58 133.35 0)
-      (effects (font (size 1.27 1.27)) (justify left))
-    )
-    (property "Footprint" "Capacitor_SMD:C_0603_1608Metric" (at 65.7352 135.89 0)
-      (effects (font (size 1.27 1.27)) hide)
-    )
-    (property "Datasheet" "~" (at 64.77 132.08 0)
-      (effects (font (size 1.27 1.27)) hide)
-    )
-    (pin "1")
-    (pin "2")
-    (instances
-      (project "minimouse"
-        (path "/d8fa4cba-2469-4231-847f-065b6b829f44/0999fad3-9a14-4ede-b729-a71c3dbbdf8e"
-          (reference "C10") (unit 1)
-        )
-      )
-    )
-  )
   (symbol (lib_id "Device:C") (at 186.69 59.69 0) (unit 1)
     (in_bom yes) (on_board yes) (dnp no) (fields_autoplaced)
@@
       (effects (font (size 1.27 1.27)))
     )
-    (property "Footprint" "" (at 80.01 92.202 90)
+    (property "Footprint" "Resistor_SMD:R_0603_1608Metric" (at 80.01 92.202 90)
       (effects (font (size 1.27 1.27)) hide)
     )
@@
     )
   )
-  (symbol (lib_id "power:+3.3V") (at 64.77 110.49 0) (unit 1)
-    (in_bom yes) (on_board yes) (dnp no) (fields_autoplaced)
-    (property "Reference" "#PWR019" (at 64.77 114.3 0)
-      (effects (font (size 1.27 1.27)) hide)
-    )
-    (property "Value" "+3.3V" (at 64.77 105.41 0)
-      (effects (font (size 1.27 1.27)))
-    )
-    (property "Footprint" "" (at 64.77 110.49 0)
-      (effects (font (size 1.27 1.27)) hide)
-    )
-    (property "Datasheet" "" (at 64.77 110.49 0)
-      (effects (font (size 1.27 1.27)) hide)
-    )
-    (pin "1")
-    (instances
-      (project "minimouse"
-        (path "/d8fa4cba-2469-4231-847f-065b6b829f44/0999fad3-9a14-4ede-b729-a71c3dbbdf8e"
-          (reference "#PWR019") (unit 1)
-        )
-      )
-    )
-  )
   (symbol (lib_id "power:+BATT") (at 22.86 107.95 0) (unit 1)
     (in_bom yes) (on_board yes) (dnp no) (fields_autoplaced)
@@
       (effects (font (size 1.27 1.27)))
     )
-    (property "Footprint" "Resistor_SMD:R_0603_1608Metric" (at 172.72 98.298 90)
+    (property "Footprint" "Resistor_SMD:R_2512_6332Metric" (at 172.72 98.298 90)
       (effects (font (size 1.27 1.27)) hide)
     )
@@
     )
   )
-  (symbol (lib_id "power:GND") (at 64.77 139.7 0) (unit 1)
-    (in_bom yes) (on_board yes) (dnp no) (fields_autoplaced)
-    (property "Reference" "#PWR020" (at 64.77 146.05 0)
-      (effects (font (size 1.27 1.27)) hide)
-    )
-    (property "Value" "GND" (at 64.77 144.78 0)
-      (effects (font (size 1.27 1.27)))
-    )
-    (property "Footprint" "" (at 64.77 139.7 0)
-      (effects (font (size 1.27 1.27)) hide)
-    )
-    (property "Datasheet" "" (at 64.77 139.7 0)
-      (effects (font (size 1.27 1.27)) hide)
-    )
-    (pin "1")
-    (instances
-      (project "minimouse"
-        (path "/d8fa4cba-2469-4231-847f-065b6b829f44/0999fad3-9a14-4ede-b729-a71c3dbbdf8e"
-          (reference "#PWR020") (unit 1)
-        )
-      )
-    )
-  )
   (symbol (lib_id "power:GND") (at 180.34 85.09 0) (unit 1)
     (in_bom yes) (on_board yes) (dnp no) (fields_autoplaced)
@@
   (symbol (lib_id "Device:R") (at 80.01 85.09 270) (unit 1)
     (in_bom yes) (on_board yes) (dnp no) (fields_autoplaced)
-    (property "Reference" "R20" (at 80.01 78.74 90)
+    (property "Reference" "R25" (at 80.01 78.74 90)
       (effects (font (size 1.27 1.27)) hide)
     )
@@
     (instances
       (project "minimouse"
-        (path "/d8fa4cba-2469-4231-847f-065b6b829f44/d17bb1c7-f68a-465e-9a17-5858ef86fc30"
-          (reference "R20") (unit 1)
-        )
         (path "/d8fa4cba-2469-4231-847f-065b6b829f44/0999fad3-9a14-4ede-b729-a71c3dbbdf8e"
           (reference "R25") (unit 1)
@@
       (effects (font (size 1.27 1.27)))
     )
-    (property "Footprint" "Resistor_SMD:R_0603_1608Metric" (at 172.72 85.598 90)
-      (effects (font (size 1.27 1.27)) hide)
-    )
+    (property "Footprint" "Resistor_SMD:R_2512_6332Metric" (at 172.72 85.598 90)
+      (effects (font (size 1.27 1.27)) hide)
+    )

Commit message: LAST TP
Parts:
- removed R25: 100, Resistor_SMD:R_0603_1608Metric, symbol Device:R
- R9: renamed from R10; value 100 -> 10k
- renumbered R11 to R10, R12 to R11, R13 to R12, R14 to R13, R15 to R14, R16 to R15
Connections:
- net FAULT: now also C8.1, R9.1, U2.13 (EN/FLT)
