File: mm_power.kicad_sch (KiCad schematic)
At the start: 1 part, among them J5 Conn_01x02

Commit message: TP2
Parts:
- added C11, C12: 1uF, Capacitor_SMD:C_0603_1608Metric, symbol Device:C
- added D1: LED, LED_SMD:LED_0603_1608Metric, symbol Device:LED
- added R18: 330, Resistor_SMD:R_0603_1608Metric, symbol Device:R
- added U3: LP5907MFX-3.3, Package_TO_SOT_SMD:SOT-23-5, symbol Regulator_Linear:LP5907MFX-3.3
Connections:
- net +BATT: now also C11.1, U3.1 (IN), U3.3 (EN)
- net GND: now also C11.2, C12.2, R18.2, U3.2 (GND)
- new net: D1.1 (K), R18.1
- new net +3.3V: C12.1, D1.2 (A), U3.5 (OUT)

Commit message: TP4
Parts:
- C11, C12: value 1uF -> 2.2uF
- D1: value LED -> ON
Connections:
- net +3.3V: now also R18.1; no longer D1.2 (A)
- net GND: now also D1.1 (K); no longer R18.2
- new net: D1.2 (A), R18.2
Other:
- moved on the sheet: D1
Changed lines of the file:
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@@
+    (stroke (width 0) (type default))
+  )
+  (wire (pts (xy 191.77 87.63) (xy 191.77 90.17))
     (stroke (width 0) (type default))
   )
@@
     (stroke (width 0) (type default))
   )
+  (wire (pts (xy 143.51 87.63) (xy 135.89 87.63))
+    (stroke (width 0) (type default))
+  )
+  (wire (pts (xy 158.75 85.09) (xy 165.1 85.09))
+    (stroke (width 0) (type default))
+  )
+  (wire (pts (xy 86.36 95.25) (xy 86.36 100.33))
+    (stroke (width 0) (type default))
+  )
+  (wire (pts (xy 95.25 95.25) (xy 86.36 95.25))
+    (stroke (width 0) (type default))
+  )
+  (wire (pts (xy 191.77 97.79) (xy 191.77 101.6))
+    (stroke (width 0) (type default))
+  )
+  (wire (pts (xy 86.36 82.55) (xy 86.36 87.63))
+    (stroke (width 0) (type default))
+  )
   (wire (pts (xy 191.77 76.2) (xy 191.77 80.01))
     (stroke (width 0) (type default))
   )
-  (wire (pts (xy 191.77 87.63) (xy 191.77 91.44))
-    (stroke (width 0) (type default))
-  )
-  (wire (pts (xy 143.51 87.63) (xy 135.89 87.63))
-    (stroke (width 0) (type default))
-  )
-  (wire (pts (xy 158.75 85.09) (xy 165.1 85.09))
-    (stroke (width 0) (type default))
-  )
-  (wire (pts (xy 86.36 95.25) (xy 86.36 100.33))
-    (stroke (width 0) (type default))
-  )
-  (wire (pts (xy 95.25 95.25) (xy 86.36 95.25))
-    (stroke (width 0) (type default))
-  )
-  (wire (pts (xy 86.36 82.55) (xy 86.36 87.63))
-    (stroke (width 0) (type default))
-  )
   (wire (pts (xy 80.01 90.17) (xy 86.36 90.17))
-    (stroke (width 0) (type default))
-  )
-  (wire (pts (xy 191.77 99.06) (xy 191.77 101.6))
     (stroke (width 0) (type default))
   )
@@
       (effects (font (size 1.27 1.27)) (justify left) hide)
     )
-    (property "Value" "1uF" (at 129.54 92.71 0)
+    (property "Value" "2.2uF" (at 129.54 92.71 0)
       (effects (font (size 1.27 1.27)) (justify left))
     )
@@
       (effects (font (size 1.27 1.27)) (justify left) hide)
     )
-    (property "Value" "1uF" (at 168.91 92.71 0)
+    (property "Value" "2.2uF" (at 168.91 92.71 0)
       (effects (font (size 1.27 1.27)) (justify left))
     )
@@
     )
   )
-  (symbol (lib_id "Device:LED") (at 191.77 83.82 90) (unit 1)
-    (in_bom yes) (on_board yes) (dnp no) (fields_autoplaced)
-    (property "Reference" "D1" (at 195.58 84.1375 90)
+  (symbol (lib_id "Device:LED") (at 191.77 93.98 90) (unit 1)
+    (in_bom yes) (on_board yes) (dnp no) (fields_autoplaced)
+    (property "Reference" "D1" (at 195.58 94.2975 90)
       (effects (font (size 1.27 1.27)) (justify right))
     )
-    (property "Value" "LED" (at 195.58 86.6775 90)
+    (property "Value" "ON" (at 195.58 96.8375 90)
       (effects (font (size 1.27 1.27)) (justify right))
     )
-    (property "Footprint" "LED_SMD:LED_0603_1608Metric" (at 191.77 83.82 0)
+    (property "Footprint" "LED_SMD:LED_0603_1608Metric" (at 191.77 93.98 0)
+      (effects (font (size 1.27 1.27)) hide)
+    )
+    (property "Datasheet" "~" (at 191.77 93.98 0)
+      (effects (font (size 1.27 1.27)) hide)
+    )
+    (pin "1")
+    (pin "2")
+    (instances
+      (project "minimouse"
+        (path "/d8fa4cba-2469-4231-847f-065b6b829f44/3f9b0845-5778-418c-a7a8-03da2392145e"
+          (reference "D1") (unit 1)
+        )
+      )
+    )
+  )
+  (symbol (lib_id "Device:R") (at 191.77 83.82 0) (unit 1)
+    (in_bom yes) (on_board yes) (dnp no) (fields_autoplaced)
+    (property "Reference" "R18" (at 194.31 82.55 0)
+      (effects (font (size 1.27 1.27)) (justify left) hide)
+    )
+    (property "Value" "330" (at 194.31 85.09 0)
+      (effects (font (size 1.27 1.27)) (justify left))
+    )
+    (property "Footprint" "Resistor_SMD:R_0603_1608Metric" (at 189.992 83.82 90)
       (effects (font (size 1.27 1.27)) hide)
     )
@@
       (effects (font (size 1.27 1.27)) hide)
     )
-    (pin "1")
-    (pin "2")
-    (instances
-      (project "minimouse"
-        (path "/d8fa4cba-2469-4231-847f-065b6b829f44/3f9b0845-5778-418c-a7a8-03da2392145e"
-          (reference "D1") (unit 1)
-        )
-      )
-    )
-  )
-  (symbol (lib_id "Device:R") (at 191.77 95.25 0) (unit 1)
-    (in_bom yes) (on_board yes) (dnp no) (fields_autoplaced)
-    (property "Reference" "R18" (at 194.31 93.98 0)
-      (effects (font (size 1.27 1.27)) (justify left) hide)
-    )
-    (property "Value" "330" (at 194.31 96.52 0)
-      (effects (font (size 1.27 1.27)) (justify left))
-    )
-    (property "Footprint" "Resistor_SMD:R_0603_1608Metric" (at 189.992 95.25 90)
-      (effects (font (size 1.27 1.27)) hide)
-    )
-    (property "Datasheet" "~" (at 191.77 95.25 0)
-      (effects (font (size 1.27 1.27)) hide)
-    )

Commit message: LAST TP
Parts:
- added 3.3V_test1, 5V_TEST1: TestPoint, TestPoint:TestPoint_Pad_D2.0mm, symbol Connector:TestPoint
- added D2: D_Zener, Diode_SMD:D_0402_1005Metric, symbol Device:D_Zener
- added Q1: Si2319CDS, Package_TO_SOT_SMD:SOT-23, symbol Transistor_FET:Si2319CDS
- added R22: 10k, Resistor_SMD:R_0603_1608Metric, symbol Device:R
- renumbered R18 to R23
Connections:
- net +3.3V: now also 3.3V_test1.1
- net +BATT: now also 5V_TEST1.1, D2.1 (K), Q1.2 (S); no longer J5.2 (Pin_2)
- net GND: now also R22.2
- new net: D2.2 (A), Q1.1 (G), R22.1
- new net: J5.2 (Pin_2), Q1.3 (D)
Other:
- moved on the sheet: J5
